File: controller-kicad/controller-kicad.kicad_sch (KiCad schematic)
At the start: 26 parts

Commit message: Started mosfets
Parts:
- added J? (x4): Conn_01x02_Female, symbol Connector:Conn_01x02_Female
- added J?: Conn_01x03_Male, symbol Connector:Conn_01x03_Male
- added U?: MCP1416, Package_TO_SOT_SMD:SOT-23-5, symbol Driver_FET:MCP1416
- added U?: IPD60R600, symbol custom_symbols:IPD60R600
Connections:
- net GND: now also J?.2 (Pin_2), J?.2 (Pin_2), J?.2 (Pin_2), J?.2 (Pin_2), J?.3 (Pin_3), U?.3 (SOURCE), U?.4 (GND)
- net +12V: now reaches U?.3 (VI)
- net +12V: now also J?.2 (Pin_2), U?.2 (Vdd)
- new net: U?.1 (GATE), U?.5 (OUT)
- new net SV1: J?.1 (Pin_1), U?.2 (DRAIN)
- new net SV1_CTRL: U?.3 (IN)
- new net SV2: J?.1 (Pin_1)
- new net SV3: J?.1 (Pin_1)
- new net SV4: J?.1 (Pin_1)
- new net Vdrive: J?.1 (Pin_1)
Other:
- moved on the sheet: J?, U?
